File: Hardware/PCBCONVEYOR.sch (EAGLE design)
At the start: 8 parts, among them J1 SPI-LCD, J11 IO, J2 I2CBR, J3 M06-PLAIN, J4 SPI-LCD, J5 I2CBR, J6 M12-PLAIN, J7 M12-PLAIN

Commit message: v1.0 release.
Parts:
- added C1, C2: 220uF, SuperHouse-Capacitors:CAP_POLCPOL-RADIAL-220UF-50V
- added D2: SS56, SuperHouse-Diodes:DIODESMA
- added D4, D5: (no value), SuperHouse-Diodes:DIODESOD
- added D7: TVSDUAL-T24CAN, SuperHouse-Diodes:TVSDUAL-T24CAN
- added H2: M02X20-2.00-P-BELOW, SuperHouse-Connectors:M02X20-2.00-P-BELOW
- added IC1: MCP23017SS, SuperHouse-ICs:MCP23017SS
- added IC3: TCAN332DR, SuperHouse-ICs:MCP2551
- added J10: SENSOR_R, SuperHouse-Connectors:M02X3-SHROUDED
- added J12: Right Output, SuperHouse-Connectors:M02-KF2510
- added J8: CAN_BUS, SuperHouse-Connectors:M04-SCREW-3.81MM-VERT-PLUG
- added J9: CAN_TERM, SuperHouse-Connectors:M02-PIN-JUMP-Y
- added K1, K2: REED-SIL, SuperHouse-Relays:REED-SIL
- added MOD1, MOD2: STEPSTICK, SuperHouse-MotorDrivers:STEPSTICK
- added OK1, OK2: LTV816-SMT, SuperHouse-LEDs:LTV816-SMT
- added Q1, Q2: 2N7002, SuperHouse-Transistors:MOSFET-NCHANNEL-233
- added R1, R11, R19, R5, R7, R9: 10K, SuperHouse-Resistors:RESISTOR0603
- added R10, R6: 560R, SuperHouse-Resistors:RESISTOR0603
- added R12, R8: 1K, SuperHouse-Resistors:RESISTOR0603
- added R2, R3: 4K7, SuperHouse-Resistors:RESISTOR0603
- added R4: 120R, SuperHouse-Resistors:RESISTOR2010
- added SW1: Power, SuperHouse-Switches:SWITCH-DPDT3
- added VR1: DC5V3A-PTH, SuperHouse-Regulators:DC5V3A-PTH
- J1: value SPI-LCD -> Limit Sensor; device SuperHouse-Connectors:M02X4-S-BELOW -> SuperHouse-Connectors:M03-PIN
- J11: value IO -> Left Output; device SuperHouse-Connectors:M08-PIN-BELOW -> SuperHouse-Connectors:M02-KF2510
- J2: value I2CBR -> (none); device SuperHouse-Connectors:M02X3-SOCKET-BELOW -> SuperHouse-Connectors:M04-SCREW-3.81MM-VERT-PLUG
- J3: value M06-PLAIN -> CAN_BUS; device SuperHouse-Connectors:M06-PLAIN -> SuperHouse-Connectors:M04-SCREW-3.81MM-VERT-PLUG
- J4: value SPI-LCD -> Left Input; device SuperHouse-Connectors:M02X4-SHROUD -> SuperHouse-Connectors:M02-KF2510
- J5: value I2CBR -> (none); device SuperHouse-Connectors:M02X3-SHROUDED -> SuperHouse-Connectors:M04-SCREW-3.81MM-VERT-PLUG
- J6: value M12-PLAIN -> Right Input; device SuperHouse-Connectors:M12-PLAIN -> SuperHouse-Connectors:M02-KF2510
- J7: value M12-PLAIN -> SENSOR_L; device SuperHouse-Connectors:M12-PLAIN -> SuperHouse-Connectors:M02X3-SHROUDED
Connections:
- removed net !RESET: J2.6, J5.6
- removed net 12V: J2.3, J5.3
- removed net IO14_TFT_BLK: J1.7, J4.7
- removed net IO16_RX2: J11.8, J3.6
- removed net IO17_TX2: J11.7, J3.5
- removed net IO18_SCLK: J1.3, J4.3
- removed net IO21_SDA: J11.3, J2.2, J3.1, J5.2
- removed net IO22_SCL: J11.4, J2.1, J3.2, J5.1
- removed net IO23_COPI: J1.4, J4.4
- removed net IO25_TFT_CS: J1.8, J4.8
- removed net IO2_TFT_DC: J1.6, J4.6
- removed net IO32_SCL2: J11.6, J3.4
- removed net IO33_SDA2: J11.5, J3.3
- removed net IO4_TFT_RST: J1.5, J4.5
- new net 5V: H2.1, H2.2, H2.39, H2.40, K11.+, K21.+, VR1.3
- new net CAN_H1: D7.2, IC3.CANH, J3.1, J8.1, R4.1
- new net CAN_L1: D7.1, IC3.CANL, J3.2, J8.2, J9.1
- new net CAN_VIN: D2.A, J3.3, J8.3
- new net ESP_EN: H2.18
- new net GPA0_XSHUT_L: D4.C, IC1.GPA0
- new net GPA1_XSHUT_R: D5.C, IC1.GPA1
- new net GPA2_!X_ENABLE: IC1.GPA2, MOD2.!ENABLE
- new net GPA3_!Y_ENABLE: IC1.GPA3, MOD1.!ENABLE
- new net GPA4_LEFT_IN: IC1.GPA4, OK1.COL, R5.1
- new net GPA5_LEFT_OUT: IC1.GPA5, R8.1
- new net GPA6_RIGHT_IN: IC1.GPA6, OK2.COL, R9.1
- new net GPA7_RIGHT_OUT: IC1.GPA7, R12.1
- new net GPB0: IC1.GPB0
- new net GPB1: IC1.GPB1
- new net GPB2: IC1.GPB2
- new net GPB3: IC1.GPB3
- new net GPB4: IC1.GPB4
- new net GPB5: IC1.GPB5
- new net GPB6: IC1.GPB6
- new net GPB7: IC1.GPB7
- new net IO0: H2.24
- new net IO12_X_STEP: H2.23, MOD2.STEP
- new net IO13_LCD_COPI: H2.16
- new net IO14_LCD_CLK: H2.25
- new net IO15_LCD_CS: H2.14
- new net IO18_I2C_SDA: H2.17, IC1.SDA, J10.4, J7.4, R2.1
- new net IO19_I2C_SCL: H2.15, IC1.SCL, J10.3, J7.3, R3.1
- new net IO2: H2.12
- new net IO21_LCD_RS: H2.19
- new net IO22_LCD_RST: H2.20
- new net IO23_LCD_BL: H2.22
- new net IO25_X_DIR: H2.28, MOD2.DIR
- new net IO26_Y_DIR: H2.30, MOD1.DIR
- new net IO27_Y_STEP: H2.27, MOD1.STEP
- new net IO32: H2.29
- new net IO33: H2.31
- new net IO34: H2.13
- new net IO35: H2.32
- new net IO36: H2.9
- new net IO39_LIMIT: H2.11, J1.3, R1.1
- new net IO4_CAN_RX: H2.10, IC3.RXD
- new net IO5_CAN_TX: H2.26, IC3.TXD
- new net N$1: J2.1, MOD2.2B
- new net N$2: IC3.RS, R19.2
- new net N$20: J9.2, R4.2
- new net N$21: J2.2, MOD2.2A
- new net N$22: D5.A, J10.6
- new net N$24: J4.1, OK1.A
- new net N$25: J5.1, MOD1.2B
- new net N$26: J4.2, R6.1
- new net N$27: D4.A, J7.6
- new net N$28: K11.-, Q1.D
- new net N$29: J5.2, MOD1.2A
- new net N$3: IC1.!RESET
- new net N$30: J5.3, MOD1.1A
- new net N$31: J11.2, K12.P
- new net N$32: Q1.G, R7.2, R8.2
- new net N$34: J11.1, K12.S
- new net N$35: J5.4, MOD1.1B
- new net N$36: Q2.G, R11.2, R12.2
- new net N$38: K21.-, Q2.D
- new net N$40: J12.2, K22.P
- new net N$41: J12.1, K22.S
- new net N$42: J6.1, OK2.A
- new net N$43: J6.2, R10.1
- new net N$44: J2.3, MOD2.1A
- new net N$45: J2.4, MOD2.1B
- new net TXD: H2.21
- new net VIN: D2.C, SW1.1, SW1.6
- new net VSWITCHED: C1.+, C2.+, MOD1.VMOT, MOD2.VMOT, R10.2, R6.2, SW1.2, SW1.5, VR1.2
- net 3.3V: now also H2.3, H2.37, H2.38, H2.4, IC1.VDD, IC3.VDD, J10.1, J7.1, MOD1.!RESET, MOD1.!SLEEP, MOD1.MS1, MOD1.MS2, MOD1.VDD, MOD2.!RESET, MOD2.!SLEEP, MOD2.MS1, MOD2.MS2, MOD2.VDD, R1.2, R2.2, R3.2, R5.2, R9.2; no longer J11.1, J2.5, J4.2, J5.5, J6.1, J6.10, J6.11, J6.12, J6.2, J6.3, J6.4, J6.5, J6.6, J6.7, J6.8, J6.9
- net GND: now also C1.-, C2.-, D7.3, H2.33, H2.34, H2.35, H2.36, H2.5, H2.6, H2.7, H2.8, IC1.A0, IC1.A1, IC1.A2, IC1.VSS, IC3.VSS, J10.2, J3.4, J8.4, MOD1.GND, MOD1.MS3, MOD2.GND, MOD2.MS3, OK1.C, OK1.EMIT, OK2.C, OK2.EMIT, Q1.S, Q2.S, R11.1, R19.1, R7.1, VR1.1, VR1.4; no longer J11.2, J2.4, J4.1, J5.4, J7.1, J7.10, J7.11, J7.12, J7.3, J7.4, J7.5, J7.6, J7.7, J7.8, J7.9
Other:
- note added: "1/8 microstepping: MS1=high MS2=high MS3=low"
- note added: "1A"
- note added: "1B"
- note added: "2A"
- note added: "2B"
- note added: "5V Regulator"
- note added: "CAN Bus Interface"
- note added: "CAN_H"
- note added: "CAN_L"
- note added: "I/O Expander"
- note added: "IO12 is a strapping pin. It must not be held high at boot. Luckily, stepper modules use active high inputs."
- note added: "Main Board Header"
- note added: "Note: TCAN332DR is used instead of MCP2551 because it can operate at 3.3V"
- note added: "PCB Sensors"
- note added: "Ready-In/Out Left"
- note added: "Ready-In/Out Right"
- note added: "SKU: WT32SC01-TEMPLATE"
- note added: "Signal"
- note added: "Use servo extension cable for limit sensor"
- note added: "VRAW"
- note added: "WT32-SC01 Conveyor Controller"
- note added: "X-Axis Stepper Driver"
- note added: "Y-Axis Limit Sensor"
- note added: "Y-Axis Stepper Driver"
- note removed: "I2CBR Passthrough"
- note removed: "IO16_RX2"
- note removed: "IO17_TX2"
- note removed: "IO21_SDA"
- note removed: "IO22_SCL"
- note removed: "IO32_SCL2"
- note removed: "IO33_SDA2"
- note removed: "LCD Passthrough"
- note removed: "Prototyping Area"
- note removed: "Rack32 I/O"
- note removed: "Rack32 Proto Expansion Board"
- note removed: "SKU: R32PROTO"
- note removed: "Top I2CBR Header"
- note removed: "Top LCD Header"
